File: keyboards/crkbd/keymaps/henry_right/adapter/trackpad.kicad_pcb (KiCad board)
At the start: 2 copper layers, 33.4 x 18.4 mm, 9 parts, among them J1 Conn_01x12, U1 Elite-C, U3 NCP1117-3.3_SOT223, U4 TXB0104D

Commit message: 배치 변경
Parts:
- moved C1 0.64 mm to (117.5, 74.3)
- moved C2 0.64 mm to (117.5, 83.8)
- moved C3 0.63 mm to (114.9, 83.8)
- moved C4 0.63 mm to (114.9, 74.3)
- moved R1 0.30 mm to (126.7, 79.1), turned to 90 degrees
- turned U4 to 90 degrees
Connections:
- U1 pad 27: LVL_SHIFT -> TP_BTN1
- U1 pad 29: TP_BTN1 -> LVL_SHIFT
- U4 pad 10: TP_DR -> PD1
- U4 pad 11: TP_BTN1 -> PD0
- U4 pad 12: PD0 -> TP_BTN1
- U4 pad 13: PD1 -> TP_DR
- U4 pad 2: TP_SDA_3V3 -> TP_DR_3V3
- U4 pad 3: TP_SCL_3V3 -> TP_BTN1_3V3
- U4 pad 4: TP_BTN1_3V3 -> TP_SCL_3V3
- U4 pad 5: TP_DR_3V3 -> TP_SDA_3V3
Changed lines of the file:
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@@
     (add_net GND)
     (add_net LVL_SHIFT)
+    (add_net "Net-(J1-Pad10)")
+    (add_net "Net-(J1-Pad11)")
+    (add_net "Net-(J1-Pad12)")
+    (add_net "Net-(J1-Pad6)")
+    (add_net "Net-(J1-Pad7)")
+    (add_net "Net-(J1-Pad8)")
+    (add_net "Net-(U1-Pad26)")
+    (add_net "Net-(U1-Pad28)")
+    (add_net "Net-(U4-Pad6)")
+    (add_net "Net-(U4-Pad9)")
+    (add_net PB0)
+    (add_net PB1)
+    (add_net PB2)
+    (add_net PB3)
+    (add_net PB4)
+    (add_net PB5)
+    (add_net PB6)
+    (add_net PC6)
     (add_net PD0)
     (add_net PD1)
+    (add_net PD2)
+    (add_net PD3)
+    (add_net PD4)
+    (add_net PD7)
+    (add_net PE6)
+    (add_net PF4)
+    (add_net PF5)
+    (add_net PF6)
+    (add_net PF7)
+    (add_net RST)
     (add_net TP_BTN1)
     (add_net TP_BTN1_3V3)
@@
     (pad 24 thru_hole circle (at -13.97 7.62) (size 1.7526 1.7526) (drill 1.0922) (layers *.Cu *.SilkS *.Mask))
     (pad 29 thru_hole circle (at 13.97 5.08) (size 1.7526 1.7526) (drill 1.0922) (layers *.Cu *.SilkS *.Mask)
-      (net 12 TP_BTN1))
+      (net 3 LVL_SHIFT))
     (pad 28 thru_hole circle (at 13.97 2.54) (size 1.7526 1.7526) (drill 1.0922) (layers *.Cu *.SilkS *.Mask))
     (pad 27 thru_hole circle (at 13.97 0) (size 1.7526 1.7526) (drill 1.0922) (layers *.Cu *.SilkS *.Mask)
-      (net 3 LVL_SHIFT))
+      (net 12 TP_BTN1))
     (pad 26 thru_hole circle (at 13.97 -2.54) (size 1.7526 1.7526) (drill 1.0922) (layers *.Cu *.SilkS *.Mask))
     (pad 25 thru_hole circle (at 13.97 -5.08) (size 1.7526 1.7526) (drill 1.0922) (layers *.Cu *.SilkS *.Mask)
@@
   )
   (module Capacitor_SMD:C_0805_2012Metric (layer B.Cu)
-    (at 115.57 83.82 270)
+    (at 114.935 83.82 270)
     (descr "Capacitor SMD 0805 (2012 Metric), square (rectangular) end terminal, IPC_7351 nominal, (Body size source: https://docs.google.com/spreadsheets/d/1BsfQQcO9C6DZCsRaXUlFlo91Tg2WpOkGARC1WS5S8t0/edit?usp=sharing), generated with kicad-footprint-generator")
     (tags capacitor)
@@
   )
   (module Capacitor_SMD:C_0805_2012Metric (layer B.Cu)
-    (at 115.57 74.295 90)
+    (at 114.935 74.295 90)
     (descr "Capacitor SMD 0805 (2012 Metric), square (rectangular) end terminal, IPC_7351 nominal, (Body size source: https://docs.google.com/spreadsheets/d/1BsfQQcO9C6DZCsRaXUlFlo91Tg2WpOkGARC1WS5S8t0/edit?usp=sharing), generated with kicad-footprint-generator")
     (tags capacitor)
@@
   )
   (module Resistor_SMD:R_0805_2012Metric (layer B.Cu)
-    (at 127 79.075 270)
+    (at 126.7 79.075 90)
     (descr "Resistor SMD 0805 (2012 Metric), square (rectangular) end terminal, IPC_7351 nominal, (Body size source: https://docs.google.com/spreadsheets/d/1BsfQQcO9C6DZCsRaXUlFlo91Tg2WpOkGARC1WS5S8t0/edit?usp=sharing), generated with kicad-footprint-generator")
     (tags resistor)
@@
       (effects (font (size 0.5 0.5) (thickness 0.08)) (justify mirror))
     )
-    (pad 1 smd roundrect (at -0.9375 0 270) (size 0.975 1.4) (layers B.Cu B.Paste B.Mask) (roundrect_rratio 0.25)
+    (pad 1 smd roundrect (at -0.9375 0 90) (size 0.975 1.4) (layers B.Cu B.Paste B.Mask) (roundrect_rratio 0.25)
       (net 3 LVL_SHIFT))
-    (pad 2 smd roundrect (at 0.9375 0 270) (size 0.975 1.4) (layers B.Cu B.Paste B.Mask) (roundrect_rratio 0.25)
+    (pad 2 smd roundrect (at 0.9375 0 90) (size 0.975 1.4) (layers B.Cu B.Paste B.Mask) (roundrect_rratio 0.25)
       (net 1 GND))
     (model ${KISYS3DMOD}/Resistor_SMD.3dshapes/R_0805_2012Metric.wrl
@@
   )
   (module Capacitor_SMD:C_0805_2012Metric (layer B.Cu)
-    (at 118.11 74.295 90)
+    (at 117.475 74.295 90)
     (descr "Capacitor SMD 0805 (2012 Metric), square (rectangular) end terminal, IPC_7351 nominal, (Body size source: https://docs.google.com/spreadsheets/d/1BsfQQcO9C6DZCsRaXUlFlo91Tg2WpOkGARC1WS5S8t0/edit?usp=sharing), generated with kicad-footprint-generator")
     (tags capacitor)
@@
   )
   (module Capacitor_SMD:C_0805_2012Metric (layer B.Cu)
-    (at 118.11 83.82 270)
+    (at 117.475 83.82 270)
     (descr "Capacitor SMD 0805 (2012 Metric), square (rectangular) end terminal, IPC_7351 nominal, (Body size source: https://docs.google.com/spreadsheets/d/1BsfQQcO9C6DZCsRaXUlFlo91Tg2WpOkGARC1WS5S8t0/edit?usp=sharing), generated with kicad-footprint-generator")
     (tags capacitor)
@@
   )
   (module Package_SO:SOIC-14_3.9x8.7mm_P1.27mm (layer B.Cu)
-    (at 109.22 79.06)
+    (at 109.22 79.06 90)
     (descr "14-Lead Plastic Small Outline (SL) - Narrow, 3.90 mm Body [SOIC] (see Microchip Packaging Specification 00000049BS.pdf)")
     (tags "SOIC 1.27")
     (attr smd)
-    (fp_text reference U4 (at 0 3.06 180) (layer B.SilkS)
-      (effects (font (size 1 1) (thickness 0.15)) (justify mirror))
-    )
-    (fp_text value TXB0104D (at 0 -5.375 180) (layer B.Fab)
-      (effects (font (size 1 1) (thickness 0.15)) (justify mirror))
-    )
-    (fp_text user %R (at 0 0 180) (layer B.Fab)
+    (fp_text reference U4 (at 0 3.06 270) (layer B.SilkS)
+      (effects (font (size 1 1) (thickness 0.15)) (justify mirror))
+    )
+    (fp_text value TXB0104D (at 0 -5.375 270) (layer B.Fab)
+      (effects (font (size 1 1) (thickness 0.15)) (justify mirror))
+    )
+    (fp_text user %R (at 0 0 270) (layer B.Fab)
       (effects (font (size 0.9 0.9) (thickness 0.135)) (justify mirror))
     )
@@
     (fp_line (start -2.075 -4.45) (end 2.075 -4.45) (layer B.SilkS) (width 0.15))
     (fp_line (start -2.075 4.425) (end -3.45 4.425) (layer B.SilkS) (width 0.15))
-    (pad 1 smd rect (at -2.7 3.81) (size 1.5 0.6) (layers B.Cu B.Paste B.Mask)
+    (pad 1 smd rect (at -2.7 3.81 90) (size 1.5 0.6) (layers B.Cu B.Paste B.Mask)
       (net 6 +3V3))
-    (pad 2 smd rect (at -2.7 2.54) (size 1.5 0.6) (layers B.Cu B.Paste B.Mask)
+    (pad 2 smd rect (at -2.7 2.54 90) (size 1.5 0.6) (layers B.Cu B.Paste B.Mask)
+      (net 9 TP_DR_3V3))
+    (pad 3 smd rect (at -2.7 1.27 90) (size 1.5 0.6) (layers B.Cu B.Paste B.Mask)
+      (net 11 TP_BTN1_3V3))
+    (pad 4 smd rect (at -2.7 0 90) (size 1.5 0.6) (layers B.Cu B.Paste B.Mask)
+      (net 8 TP_SCL_3V3))
+    (pad 5 smd rect (at -2.7 -1.27 90) (size 1.5 0.6) (layers B.Cu B.Paste B.Mask)
       (net 7 TP_SDA_3V3))
-    (pad 3 smd rect (at -2.7 1.27) (size 1.5 0.6) (layers B.Cu B.Paste B.Mask)
-      (net 8 TP_SCL_3V3))
-    (pad 4 smd rect (at -2.7 0) (size 1.5 0.6) (layers B.Cu B.Paste B.Mask)
-      (net 11 TP_BTN1_3V3))
-    (pad 5 smd rect (at -2.7 -1.27) (size 1.5 0.6) (layers B.Cu B.Paste B.Mask)
-      (net 9 TP_DR_3V3))
-    (pad 6 smd rect (at -2.7 -2.54) (size 1.5 0.6) (layers B.Cu B.Paste B.Mask))
-    (pad 7 smd rect (at -2.7 -3.81) (size 1.5 0.6) (layers B.Cu B.Paste B.Mask)
-      (net 1 GND))
-    (pad 8 smd rect (at 2.7 -3.81) (size 1.5 0.6) (layers B.Cu B.Paste B.Mask)
+    (pad 6 smd rect (at -2.7 -2.54 90) (size 1.5 0.6) (layers B.Cu B.Paste B.Mask))
+    (pad 7 smd rect (at -2.7 -3.81 90) (size 1.5 0.6) (layers B.Cu B.Paste B.Mask)
+      (net 1 GND))
+    (pad 8 smd rect (at 2.7 -3.81 90) (size 1.5 0.6) (layers B.Cu B.Paste B.Mask)
       (net 3 LVL_SHIFT))
-    (pad 9 smd rect (at 2.7 -2.54) (size 1.5 0.6) (layers B.Cu B.Paste B.Mask))
-    (pad 10 smd rect (at 2.7 -1.27) (size 1.5 0.6) (layers B.Cu B.Paste B.Mask)
+    (pad 9 smd rect (at 2.7 -2.54 90) (size 1.5 0.6) (layers B.Cu B.Paste B.Mask))
+    (pad 10 smd rect (at 2.7 -1.27 90) (size 1.5 0.6) (layers B.Cu B.Paste B.Mask)
+      (net 5 PD1))
+    (pad 11 smd rect (at 2.7 0 90) (size 1.5 0.6) (layers B.Cu B.Paste B.Mask)
+      (net 4 PD0))
+    (pad 12 smd rect (at 2.7 1.27 90) (size 1.5 0.6) (layers B.Cu B.Paste B.Mask)
+      (net 12 TP_BTN1))
+    (pad 13 smd rect (at 2.7 2.54 90) (size 1.5 0.6) (layers B.Cu B.Paste B.Mask)
       (net 10 TP_DR))
-    (pad 11 smd rect (at 2.7 0) (size 1.5 0.6) (layers B.Cu B.Paste B.Mask)
-      (net 12 TP_BTN1))
-    (pad 12 smd rect (at 2.7 1.27) (size 1.5 0.6) (layers B.Cu B.Paste B.Mask)
-      (net 4 PD0))
-    (pad 13 smd rect (at 2.7 2.54) (size 1.5 0.6) (layers B.Cu B.Paste B.Mask)
-      (net 5 PD1))
-    (pad 14 smd rect (at 2.7 3.81) (size 1.5 0.6) (layers B.Cu B.Paste B.Mask)
+    (pad 14 smd rect (at 2.7 3.81 90) (size 1.5 0.6) (layers B.Cu B.Paste B.Mask)
       (net 2 +5V))
     (model ${KISYS3DMOD}/Package_SO.3dshapes/SOIC-14_3.9x8.7mm_P1.27mm.wrl

Commit message: 전체
Parts:
- moved C1 1.91 mm to (119.4, 74.3), turned to 0 degrees
- moved C2 1.91 mm to (119.4, 83.8), turned to 0 degrees
- moved C3 0.63 mm to (115.6, 83.8), turned to 180 degrees
- moved C4 0.63 mm to (115.6, 74.3), turned to 180 degrees
Routing:
- net +5V: track 0.00 -> 34.8 mm, vias 0 -> 4
- net LVL_SHIFT: track 0.00 -> 29.4 mm
- net +3V3: track 0.00 -> 27.3 mm
- net TP_BTN1: track 0.00 -> 21.8 mm
- net TP_DR: track 0.00 -> 20.1 mm
- net TP_DR_3V3: track 0.00 -> 11.5 mm
- net TP_BTN1_3V3: track 0.00 -> 9.39 mm
- net TP_SCL_3V3: track 0.00 -> 7.96 mm
- net PD0: track 0.00 -> 7.39 mm
- net GND: track 0.00 -> 7.39 mm, vias 0 -> 18
- net TP_SDA_3V3: track 0.00 -> 6.52 mm
- net PD1: track 0.00 -> 6.51 mm
